File: Sketches/Brug sketches/Brug sketches.kicad_sch (KiCad schematic)
At the start: 31 parts, among them M1 Motor_DC, Q1 BC547, Q2 BC547, Q3 BC547, Q4 BC547, Q5 PNP, Q6 PNP, Q7 NPN, Q8 NPN

Commit message: laatste versie 13-10-2023
Parts:
- added C? (x3): 100n, symbol core-rescue:C
- added C? (x2): 22pF, symbol core-rescue:C
- added C?: 100nF, symbol core-rescue:C
- added IC?: ATMEGA2560-A, TQFP100, symbol core-rescue:ATMEGA2560-A
- added R?: R, symbol core-rescue:R
- added R?: 1M, symbol core-rescue:R
- added Y?: 16MHz, symbol core-rescue:Crystal
Connections:
- net GND: now also C?.2, C?.2, C?.2, C?.2, C?.2, C?.2, IC?.11 (GND), IC?.32 (GND), IC?.81 (GND), IC?.99 (GND)
- net VCC: now also C?.1, C?.1, C?.1, IC?.10 (VCC), IC?.100 (AVCC), IC?.31 (VCC), IC?.80 (VCC); no longer R10.2, R11.2, R12.2, R13.2, R14.2
- new net: IC?.34 (XTAL1), R?.1
- new net: C?.1, R?.2, R?.2, Y?.2
- new net: C?.1, IC?.33 (XTAL2), R?.1, Y?.1
- new net: C?.1, IC?.98 (AREF)
- new net 50: R12.2
- new net 51: R11.2, R14.2
- new net 53: R10.2, R13.2
- new net MISO: IC?.22 ((PCINT3/MISO)PB3)
- new net MOSI: IC?.21 ((PCINT2/MOSI)PB2)
- new net RESET: IC?.30 (~{RESET})
- new net RX0: IC?.2 ((PCINT8/RXD0)PE0)
- new net SCK: IC?.20 ((PCINT1/SCK)PB1)
- new net SCL: IC?.43 ((SCL/INT0)PD0)
- new net SDA: IC?.44 ((SDA/INT1)PD1)
- new net TCK: IC?.93 ((TCK/ADC4)PF4)
- new net TDI: IC?.90 ((TDI/ADC7)PF7)
- new net TDO: IC?.91 ((TD0/ADC6)PF6)
- new net TMS: IC?.92 ((TMS/ADC5)PF5)
- new net TX0: IC?.3 ((TXD0)PE1)
Other:
- added sheet Atmega 2560 (atmega2560.kicad_sch)
