File: Sketches/Brug sketches/bruglichten.kicad_sch (KiCad schematic)
At the start: 10 parts

Commit message: laatste versie 13-10-2023
Parts:
- removed D1, D4: LED Rood, symbol Device:LED
- removed D2: LED Geel, symbol Device:LED
- removed D3, D5: LED Groen, symbol Device:LED
- removed R1, R2, R3, R4, R5: 230R, symbol Device:R
- added D10, D13: LED Rood, symbol Device:LED
- added D11, D14: LED Groen, symbol Device:LED
- added D12: LED Geel, symbol Device:LED
- added R10, R11, R12, R13, R14: 230R, symbol Device:R
Connections:
- net GND: now also D10.1 (K), D11.1 (K), D12.1 (K), D13.1 (K), D14.1 (K)
- new net: D13.2 (A), R13.1
- new net: D11.2 (A), R11.1
- new net: D14.2 (A), R14.1
- new net: D12.2 (A), R12.1
- new net: D10.2 (A), R10.1
- new net 50: R12.2
- new net 51: R11.2, R14.2
- new net 53: R10.2, R13.2
